File: hardware/NosLed.kicad_sch (KiCad schematic)
At the start: 5 parts, among them J101 LOAD, J102 PWM, J201 AC, U102 PC817

Commit message: AC Input
Parts:
- removed R101: 330R, Resistor_THT:R_Axial_DIN0207_L6.3mm_D2.5mm_P7.62mm_Horizontal, symbol Device:R
- removed U102: PC817, Package_DIP:DIP-4_W7.62mm, symbol Isolator:PC817
- added J103, J104: 380OUT, TerminalBlock_Phoenix:TerminalBlock_Phoenix_MKDS-1,5-2-5.08_1x02_P5.08mm_Horizontal, symbol Connector:Screw_Terminal_01x02
- renumbered J201 to J101, J101 to J105
Connections:
- net BP2876D/HI_GND is gone; now on net BP2876D/PWM: J102.1 (Pin_1)
- net BP2876D/PWM: no longer J102.2 (Pin_2)
- net BP2876D/AC_L renamed ACInput/AC_N
- net BP2876D/AC_N renamed ACInput/AC_L
- new net ACInput/380V: J103.1 (Pin_1), J104.2 (Pin_2)
- new net ACInput/GND: J102.2 (Pin_2), J103.2 (Pin_2), J104.1 (Pin_1)
Other:
- sheet BP2876 renamed BP2876D
- added sheet ACInput (ACInput.kicad_sch)
- sheet BP2876D ports: added 380V, GND; removed AC_L, AC_N, HI_GND
- moved on the sheet: J101, J102
