File: hardware/BP2876.kicad_sch (KiCad schematic)
At the start: 18 parts, among them U101 BP2876

Commit message: AC Input
Parts:
- removed C202: 10uF 63v, Capacitor_THT:CP_Radial_D5.0mm_P2.50mm, symbol Device:C_Polarized
- removed C204: 33uF 400v, Capacitor_THT:CP_Radial_D13.0mm_P5.00mm, symbol Device:C_Polarized
- removed D201: MB10S, Package_DIP:DIP-4_W7.62mm, symbol Diode_Bridge:MB6S
- removed F201: Fuse, Fuse:Fuseholder_Cylinder-5x20mm_Stelvio-Kontek_PTF78_Horizontal_Open, symbol Device:Fuse
- removed NT202: NetTie_2, NetTie:NetTie-2_SMD_Pad0.5mm, symbol Device:NetTie_2
- removed R204: 51K, Resistor_THT:R_Axial_DIN0207_L6.3mm_D2.5mm_P7.62mm_Horizontal, symbol Device:R
- removed RV201: 10D471, Varistor:RV_Disc_D12mm_W4.8mm_P7.5mm, symbol Device:Varistor
- added NT303: NetTie_2, NetTie:NetTie-2_SMD_Pad0.5mm, symbol Device:NetTie_2
- C302: renamed from C203; value 10uF 63v -> 10uF 100v; footprint Capacitor_THT:CP_Radial_D5.0mm_P2.50mm -> Capacitor_THT:CP_Radial_D6.3mm_P2.50mm
- R301: renamed from R202; footprint Resistor_THT:R_Axial_DIN0207_L6.3mm_D2.5mm_P7.62mm_Horizontal -> Resistor_THT:R_Axial_DIN0309_L9.0mm_D3.2mm_P12.70mm_Horizontal
- R302: renamed from R203; value 10K -> 27K
- renumbered C201 to C301, D202 to D301, L201 to L301, NT201 to NT301, NT203 to NT302, R201 to R304, R205 to R305, U101 to U301
Connections:
- net LOAD-: now also C302.2
- net at C301.2, R302.2: now also NT302.1; no longer NT302.2, U301.1 (GND)
- net LOAD+ renamed 380V
- net PWR_GND renamed GND
- net GND: now also NT302.2, NT303.1; no longer NT302.1
- new net: NT303.2, U301.1 (GND)
Other:
- moved on the sheet: C301, C302, D301, NT301, NT302, R301, R302, R305

Commit message: LNK302PN
Parts:
- renumbered NT302 to NT301, NT301 to NT302, R304 to R303, R305 to R304
Changed lines of the file:
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@@
-	)
-	(symbol
-		(lib_id "Device:R")
-		(at 166.37 85.09 270)
-		(unit 1)
-		(exclude_from_sim no)
-		(in_bom yes)
-		(on_board yes)
-		(dnp no)
-		(property "Reference" "R302"
-			(at 168.402 80.264 90)
-			(effects
-				(font
-					(size 1.27 1.27)
-				)
-				(justify right)
-			)
-		)
-		(property "Value" "27K"
-			(at 168.148 82.55 90)
-			(effects
-				(font
-					(size 1.27 1.27)
-				)
-				(justify right)
-			)
-		)
-		(property "Footprint" "Resistor_THT:R_Axial_DIN0207_L6.3mm_D2.5mm_P7.62mm_Horizontal"
-			(at 166.37 83.312 90)
-			(effects
-				(font
-					(size 1.27 1.27)
-				)
-				(hide yes)
-			)
-		)
-		(property "Datasheet" "~"
-			(at 166.37 85.09 0)
-			(effects
-				(font
-					(size 1.27 1.27)
-				)
-				(hide yes)
-			)
-		)
-		(property "Description" "Resistor"
-			(at 166.37 85.09 0)
-			(effects
-				(font
-					(size 1.27 1.27)
-				)
-				(hide yes)
-			)
-		)
-		(pin "2"
-		)
-		(pin "1"
-		)
-		(instances
-			(project "NosLed"
-				(path "/473a9690-2801-417b-8084-b7ef486d51ca/60f11f86-c817-4eb5-9dbe-13279180a35c"
-					(reference "R302")
-					(unit 1)
-				)
-			)
-		)
 	)
 	(symbol
@@
 	)
 	(symbol
+		(lib_id "Device:R")
+		(at 166.37 85.09 270)
+		(unit 1)
+		(exclude_from_sim no)
+		(in_bom yes)
+		(on_board yes)
+		(dnp no)
+		(property "Reference" "R302"
+			(at 168.402 80.264 90)
+			(effects
+				(font
+					(size 1.27 1.27)
+				)
+				(justify right)
+			)
+		)
+		(property "Value" "27K"
+			(at 168.148 82.55 90)
+			(effects
+				(font
+					(size 1.27 1.27)
+				)
+				(justify right)
+			)
+		)
+		(property "Footprint" "Resistor_THT:R_Axial_DIN0207_L6.3mm_D2.5mm_P7.62mm_Horizontal"
+			(at 166.37 83.312 90)
+			(effects
+				(font
+					(size 1.27 1.27)
+				)
+				(hide yes)
+			)
+		)
+		(property "Datasheet" "~"
+			(at 166.37 85.09 0)
+			(effects
+				(font
+					(size 1.27 1.27)
+				)
+				(hide yes)
+			)
+		)
+		(property "Description" "Resistor"
+			(at 166.37 85.09 0)
+			(effects
+				(font
+					(size 1.27 1.27)
+				)
+				(hide yes)
+			)
+		)
+		(pin "2"
+		)
+		(pin "1"
+		)
+		(instances
+			(project "NosLed"
+				(path "/473a9690-2801-417b-8084-b7ef486d51ca/60f11f86-c817-4eb5-9dbe-13279180a35c"
+					(reference "R302")
+					(unit 1)
+				)
+			)
+		)
+	)
+	(symbol
 		(lib_id "Device:NetTie_2")
 		(at 154.94 57.15 90)
@@
 		(dnp no)
 		(fields_autoplaced yes)
-		(property "Reference" "NT301"
+		(property "Reference" "NT302"
 			(at 156.21 55.8799 90)
 			(effects
@@
 			(project ""
 				(path "/473a9690-2801-417b-8084-b7ef486d51ca/60f11f86-c817-4eb5-9dbe-13279180a35c"
-					(reference "NT301")
+					(reference "NT302")
 					(unit 1)
 				)
@@
 		(on_board yes)
 		(dnp no)
-		(property "Reference" "R305"
+		(property "Reference" "R304"
 			(at 233.934 60.198 90)
 			(effects
@@
 			(project "NosLed"
 				(path "/473a9690-2801-417b-8084-b7ef486d51ca/60f11f86-c817-4eb5-9dbe-13279180a35c"
-					(reference "R305")
+					(reference "R304")
 					(unit 1)
 				)
@@
 		(dnp no)
 		(fields_autoplaced yes)
-		(property "Reference" "NT302"
+		(property "Reference" "NT301"
 			(at 148.59 80.01 0)
 			(effects
@@
 			(project "NosLed"
 				(path "/473a9690-2801-417b-8084-b7ef486d51ca/60f11f86-c817-4eb5-9dbe-13279180a35c"
-					(reference "NT302")
+					(reference "NT301")
 					(unit 1)
 				)
@@
 		(on_board yes)
 		(dnp no)
-		(property "Reference" "R304"
+		(property "Reference" "R303"
 			(at 205.994 92.964 90)
 			(effects
@@
 			(project ""
 				(path "/473a9690-2801-417b-8084-b7ef486d51ca/60f11f86-c817-4eb5-9dbe-13279180a35c"
-					(reference "R304")
-					(unit 1)
-				)
+					(reference "R303")
+					(unit 1)
+				)

Commit message: BP2956XS
Parts:
- U301: Datasheet CN https://taoic.oss-cn-hangzhou.aliyuncs.com/9208/product/HZD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 -> (none)
Changed lines of the file:
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@@
 	(generator_version "9.0")
 	(paper "A4")
+	(text_box "Rcs = Vref / I = 0.3V / 0.110A = 2.72 Ohm -> 2.7 Ohm\nRovp = (Vovp * Rcs) / (Kovp * L) = (75V * 2.7Ohm) / (5 * 0.0022H) = 18409 Ohm -> 18 kOhm"
+		(exclude_from_sim no)
+		(at 50.8 177.8 0)
+		(size 111.76 6.35)
+		(margins 0.9525 0.9525 0.9525 0.9525)
+		(stroke
+			(width -0.0001)
+			(type solid)
+		)
+		(fill
+			(type none)
+		)
+		(effects
+			(font
+				(size 1.27 1.27)
+			)
+			(justify left top)
+		)
+	)
 	(junction
 		(at 238.76 69.85)
@@
 			)
 		)
-		(property "Datasheet" "kicad-embed://BP2876D.PDF"
+		(property "Datasheet" "https://taoic.oss-cn-hangzhou.aliyuncs.com/9208/product/HZDZ88_1636526643000.pdf"
 			(at 198.882 74.168 0)
 			(effects
@@
 			(effects
 				(font
-					(size 1.27 1.27)
-				)
-				(hide yes)
-			)
-		)
-		(property "Datasheet CN" "https://taoic.oss-cn-hangzhou.aliyuncs.com/9208/product/HZDZ88_1636526643000.pdf"
-			(at 199.898 103.124 0)
-			(effects
-				(font

Commit message: Prototype
Connections:
- net 380V renamed 325V
Changed lines of the file:
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@@
 		)
 	)
-	(hierarchical_label "380V"
+	(hierarchical_label "325V"
 		(shape input)
 		(at 140.97 52.07 180)
