File: hardware/BP2956XS.kicad_sch (KiCad schematic)
At the start: 9 parts, among them U502 BP2956XS

Commit message: BP2956XS
Parts:
- removed NT501, NT503: NetTie_2, NetTie:NetTie-2_SMD_Pad0.5mm, symbol Device:NetTie_2
- R502: value 27K -> 7K5
- R503: value 3R3 -> 2R7
- U502: footprint Package_SO:SOIC-8_5.3x5.3mm_P1.27mm -> Package_DIP:DIP-8_W7.62mm
Connections:
- net GND: now also R502.2, U502.2 (GND)
Changed lines of the file:
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@@
 	(generator_version "9.0")
 	(paper "A4")
+	(text_box "Rcs = Vref / I = 0.3V / 0.110A = 2.7Ohm\nRovp = (Vovp * Rcs) / (Kovp * L) = (75v * 2.7Ohm) / (12.5 * 0.0022H) = 7360Ohm ~> 7.5KOhm"
+		(exclude_from_sim no)
+		(at 62.23 135.89 0)
+		(size 111.76 6.35)
+		(margins 0.9525 0.9525 0.9525 0.9525)
+		(stroke
+			(width -0.0001)
+			(type solid)
+		)
+		(fill
+			(type none)
+		)
+		(effects
+			(font
+				(size 1.27 1.27)
+			)
+			(justify left top)
+		)
+	)
 	(junction
 		(at 109.22 66.04)
@@
 	(wire
 		(pts
-			(xy 77.47 99.06) (xy 88.9 99.06)
-		)
-		(stroke
-			(width 0)
-			(type default)
-		)
-	)
-	(wire
-		(pts
 			(xy 127 87.63) (xy 127 99.06)
 		)
@@
 	(wire
 		(pts
-			(xy 64.77 99.06) (xy 72.39 99.06)
+			(xy 64.77 99.06) (xy 88.9 99.06)
 		)
 		(stroke
@@
 	(wire
 		(pts
-			(xy 109.22 119.38) (xy 109.22 120.65)
+			(xy 109.22 113.03) (xy 109.22 120.65)
 		)
 		(stroke
@@
 		(pts
 			(xy 139.7 83.82) (xy 139.7 88.9)
-		)
-		(stroke
-			(width 0)
-			(type default)
-		)
-	)
-	(wire
-		(pts
-			(xy 109.22 113.03) (xy 109.22 114.3)
 		)
 		(stroke
@@
 	(label "DRAIN"
 		(at 139.7 99.06 0)
-		(effects
-			(font
-				(size 1.27 1.27)
-			)
-			(justify left bottom)
-		)
-	)
-	(label "PWR_GND"
-		(at 139.7 107.95 0)
 		(effects
 			(font
@@
 				(path "/473a9690-2801-417b-8084-b7ef486d51ca/62dae79f-20f1-42ce-ac91-8f6732a4f040"
 					(reference "L501")
-					(unit 1)
-				)
-			)
-		)
-	)
-	(symbol
-		(lib_id "Device:NetTie_2")
-		(at 74.93 99.06 180)
-		(unit 1)
-		(exclude_from_sim no)
-		(in_bom no)
-		(on_board yes)
-		(dnp no)
-		(fields_autoplaced yes)
-		(property "Reference" "NT501"
-			(at 74.93 93.98 0)
-			(effects
-				(font
-					(size 1.27 1.27)
-				)
-			)
-		)
-		(property "Value" "NetTie_2"
-			(at 74.93 96.52 0)
-			(effects
-				(font
-					(size 1.27 1.27)
-				)
-			)
-		)
-		(property "Footprint" "NetTie:NetTie-2_SMD_Pad0.5mm"
-			(at 74.93 99.06 0)
-			(effects
-				(font
-					(size 1.27 1.27)
-				)
-				(hide yes)
-			)
-		)
-		(property "Datasheet" "~"
-			(at 74.93 99.06 0)
-			(effects
-				(font
-					(size 1.27 1.27)
-				)
-				(hide yes)
-			)
-		)
-		(property "Description" "Net tie, 2 pins"
-			(at 74.93 99.06 0)
-			(effects
-				(font
-					(size 1.27 1.27)
-				)
-				(hide yes)
-			)
-		)
-		(pin "1"
-		)
-		(pin "2"
-		)
-		(instances
-			(project "NosLed"
-				(path "/473a9690-2801-417b-8084-b7ef486d51ca/62dae79f-20f1-42ce-ac91-8f6732a4f040"
-					(reference "NT501")
 					(unit 1)
 				)
@@
 			)
 		)
-		(property "Footprint" "Package_SO:SOIC-8_5.3x5.3mm_P1.27mm"
+		(property "Footprint" "Package_DIP:DIP-8_W7.62mm"
 			(at 131.318 91.186 0)
 			(effects
@@
 			)
 		)
-		(property "Datasheet" "kicad-embed://1716788106817.pdf"
+		(property "Datasheet" "kicad-embed://DDWDZ123_1694244723000.pdf"
 			(at 125.222 88.138 0)
 			(effects
@@
 				(path "/473a9690-2801-417b-8084-b7ef486d51ca/62dae79f-20f1-42ce-ac91-8f6732a4f040"
 					(reference "U502")
-					(unit 1)
-				)
-			)
-		)
-	)
-	(symbol
-		(lib_id "Device:NetTie_2")
-		(at 109.22 116.84 90)
-		(unit 1)
-		(exclude_from_sim no)
-		(in_bom no)
-		(on_board yes)
-		(dnp no)
-		(fields_autoplaced yes)
-		(property "Reference" "NT503"
-			(at 110.49 115.5699 90)
-			(effects
-				(font
-					(size 1.27 1.27)
-				)
-				(justify right)
-			)
-		)
-		(property "Value" "NetTie_2"
-			(at 110.49 118.1099 90)
-			(effects
-				(font
-					(size 1.27 1.27)
-				)
-				(justify right)
-			)
-		)
-		(property "Footprint" "NetTie:NetTie-2_SMD_Pad0.5mm"
-			(at 109.22 116.84 0)
-			(effects
-				(font
-					(size 1.27 1.27)
-				)
-				(hide yes)
-			)
-		)
-		(property "Datasheet" "~"
-			(at 109.22 116.84 0)
-			(effects
-				(font
-					(size 1.27 1.27)
-				)
-				(hide yes)
-			)
-		)
-		(property "Description" "Net tie, 2 pins"
-			(at 109.22 116.84 0)
-			(effects
-				(font
-					(size 1.27 1.27)
-				)
-				(hide yes)
-			)
-		)
-		(pin "1"
-		)
-		(pin "2"
-		)
-		(instances
-			(project "NosLed"
-				(path "/473a9690-2801-417b-8084-b7ef486d51ca/62dae79f-20f1-42ce-ac91-8f6732a4f040"
-					(reference "NT503")
 					(unit 1)
 				)
@@
 			)
 		)
-		(property "Value" "3R3"
+		(property "Value" "2R7"
 			(at 132.334 109.474 90)
 			(effects
@@
 			)
 		)
-		(property "Value" "27K"
+		(property "Value" "7K5"
 			(at 94.488 96.52 90)
 			(effects

Commit message: Prototype
Parts:
- removed D501: UF4007, Diode_THT:D_DO-41_SOD81_P7.62mm_Horizontal, symbol Device:D
- added D502: US1M, Diode_SMD:D_SMA, symbol Diode:US1M
- C501: renamed from C502; footprint Capacitor_THT:CP_Radial_D6.3mm_P2.50mm -> Capacitor_THT:CP_Radial_D10.0mm_P5.00mm
- R501: renamed from R502; footprint Resistor_THT:R_Axial_DIN0207_L6.3mm_D2.5mm_P7.62mm_Horizontal -> Resistor_SMD:R_0805_2012Metric_Pad1.20x1.40mm_HandSolder
- R502: renamed from R503; footprint Resistor_THT:R_Axial_DIN0309_L9.0mm_D3.2mm_P12.70mm_Horizontal -> Resistor_SMD:R_1206_3216Metric_Pad1.30x1.75mm_HandSolder
- R503: renamed from R504; footprint Resistor_THT:R_Axial_DIN0207_L6.3mm_D2.5mm_P7.62mm_Horizontal -> Resistor_SMD:R_1206_3216Metric_Pad1.30x1.75mm_HandSolder
- U502: footprint Package_DIP:DIP-8_W7.62mm -> Package_SO:SOIC-8_5.3x5.3mm_P1.27mm
Connections:
- net DRAIN: now also D502.2 (A)
- net 380V renamed 325V
- net 325V: now also D502.1 (K)
Changed lines of the file:
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@@
 		)
 	)
-	(hierarchical_label "380V"
+	(hierarchical_label "325V"
 		(shape input)
 		(at 67.31 66.04 180)
@@
 			)
 		)
-		(property "Footprint" "Package_DIP:DIP-8_W7.62mm"
+		(property "Footprint" "Package_SO:SOIC-8_5.3x5.3mm_P1.27mm"
 			(at 131.318 91.186 0)
 			(effects
@@
 			)
 		)
-		(property "Datasheet" "kicad-embed://DDWDZ123_1694244723000.pdf"
+		(property "Datasheet" "kicad-embed://1716788106817.pdf"
 			(at 125.222 88.138 0)
 			(effects
@@
 			)
 		)
+		(pin "4"
+		)
+		(pin "3"
+		)
+		(pin "8"
+		)
+		(pin "2"
+		)
+		(pin "5"
+		)
 		(pin "6"
 		)
-		(pin "4"
-		)
-		(pin "3"
-		)
 		(pin "1"
 		)
 		(pin "7"
 		)
-		(pin "5"
-		)
-		(pin "2"
-		)
-		(pin "8"
-		)
 		(instances
 			(project ""
 				(path "/473a9690-2801-417b-8084-b7ef486d51ca/62dae79f-20f1-42ce-ac91-8f6732a4f040"
 					(reference "U502")
+					(unit 1)
+				)
+			)
+		)
+	)
+	(symbol
+		(lib_id "Diode:US1M")
+		(at 127 83.82 270)
+		(unit 1)
+		(exclude_from_sim no)
+		(in_bom yes)
+		(on_board yes)
+		(dnp no)
+		(fields_autoplaced yes)
+		(property "Reference" "D502"
+			(at 129.54 82.5499 90)
+			(effects
+				(font
+					(size 1.27 1.27)
+				)
+				(justify left)
+			)
+		)
+		(property "Value" "US1M"
+			(at 129.54 85.0899 90)
+			(effects
+				(font
+					(size 1.27 1.27)
+				)
+				(justify left)
+			)
+		)
+		(property "Footprint" "Diode_SMD:D_SMA"
+			(at 122.555 83.82 0)
+			(effects
+				(font
+					(size 1.27 1.27)
+				)
+				(hide yes)
+			)
+		)
+		(property "Datasheet" "https://www.diodes.com/assets/Datasheets/ds16008.pdf"
+			(at 127 83.82 0)
+			(effects
+				(font
+					(size 1.27 1.27)
+				)
+				(hide yes)
+			)
+		)
+		(property "Description" "1000V, 1A, General Purpose Rectifier Diode, SMA(DO-214AC)"
+			(at 127 83.82 0)
+			(effects
+				(font
+					(size 1.27 1.27)
+				)
+				(hide yes)
+			)
+		)
+		(property "Sim.Device" "D"
+			(at 127 83.82 0)
+			(effects
+				(font
+					(size 1.27 1.27)
+				)
+				(hide yes)
+			)
+		)
+		(property "Sim.Pins" "1=K 2=A"
+			(at 127 83.82 0)
+			(effects
+				(font
+					(size 1.27 1.27)
+				)
+				(hide yes)
+			)
+		)
+		(pin "2"
+		)
+		(pin "1"
+		)
+		(instances
+			(project ""
+				(path "/473a9690-2801-417b-8084-b7ef486d51ca/62dae79f-20f1-42ce-ac91-8f6732a4f040"
+					(reference "D502")
 					(unit 1)
 				)
@@
 		(dnp no)
 		(fields_autoplaced yes)
-		(property "Reference" "C502"
+		(property "Reference" "C501"
 			(at 143.51 74.0409 0)
 			(effects
@@
 			)
 		)
-		(property "Footprint" "Capacitor_THT:CP_Radial_D6.3mm_P2.50mm"
+		(property "Footprint" "Capacitor_THT:CP_Radial_D10.0mm_P5.00mm"
 			(at 140.6652 80.01 0)
 			(effects
@@
 			(project "NosLed"
 				(path "/473a9690-2801-417b-8084-b7ef486d51ca/62dae79f-20f1-42ce-ac91-8f6732a4f040"
-					(reference "C502")
+					(reference "C501")
 					(unit 1)
 				)
@@
 		(on_board yes)
 		(dnp no)
-		(property "Reference" "R503"
+		(property "Reference" "R502"
 			(at 132.334 106.934 90)
 			(effects
@@
 			)
 		)
-		(property "Footprint" "Resistor_THT:R_Axial_DIN0309_L9.0mm_D3.2mm_P12.70mm_Horizontal"
+		(property "Footprint" "Resistor_SMD:R_1206_3216Metric_Pad1.30x1.75mm_HandSolder"
 			(at 132.08 102.362 90)
 			(effects
@@
 			(project "NosLed"
 				(path "/473a9690-2801-417b-8084-b7ef486d51ca/62dae79f-20f1-42ce-ac91-8f6732a4f040"
-					(reference "R503")
+					(reference "R502")
 					(unit 1)
 				)
@@
 		(on_board yes)
 		(dnp no)
-		(property "Reference" "R502"
+		(property "Reference" "R501"
 			(at 94.742 94.234 90)
 			(effects
@@
 			)
 		)
-		(property "Footprint" "Resistor_THT:R_Axial_DIN0207_L6.3mm_D2.5mm_P7.62mm_Horizontal"
+		(property "Footprint" "Resistor_SMD:R_0805_2012Metric_Pad1.20x1.40mm_HandSolder"
 			(at 92.71 97.282 90)
 			(effects
@@
 			(project "NosLed"
 				(path "/473a9690-2801-417b-8084-b7ef486d51ca/62dae79f-20f1-42ce-ac91-8f6732a4f040"
-					(reference "R502")
+					(reference "R501")
 					(unit 1)
 				)
@@
 		(lib_id "Device:R")
 		(at 165.1 76.2 0)
-		(unit 1)
-		(exclude_from_sim no)
-		(in_bom yes)
-		(on_board yes)
-		(dnp no)
-		(property "Reference" "R504"
-			(at 160.274 74.168 90)
+		(mirror y)
+		(unit 1)
+		(exclude_from_sim no)
+		(in_bom yes)
+		(on_board yes)
+		(dnp no)
+		(property "Reference" "R503"
+			(at 169.926 74.168 90)
 			(effects
 				(font
@@
 		)
 		(property "Value" "100К"
-			(at 162.56 74.422 90)
+			(at 167.64 74.422 90)
 			(effects
 				(font
@@
 			)
 		)
-		(property "Footprint" "Resistor_THT:R_Axial_DIN0207_L6.3mm_D2.5mm_P7.62mm_Horizontal"
-			(at 163.322 76.2 90)
+		(property "Footprint" "Resistor_SMD:R_1206_3216Metric_Pad1.30x1.75mm_HandSolder"
+			(at 166.878 76.2 90)
 			(effects
 				(font
@@
 			(project "NosLed"
 				(path "/473a9690-2801-417b-8084-b7ef486d51ca/62dae79f-20f1-42ce-ac91-8f6732a4f040"
-					(reference "R504")
-					(unit 1)
-				)
-			)
-		)
-	)
-	(symbol
-		(lib_id "Device:D")
-		(at 127 83.82 270)
-		(unit 1)
-		(exclude_from_sim no)
-		(in_bom yes)
-		(on_board yes)
-		(dnp no)
-		(property "Reference" "D501"
-			(at 132.08 85.09 90)
-			(effects
-				(font
-					(size 1.27 1.27)
-				)
-			)
-		)
-		(property "Value" "UF4007"
-			(at 132.08 82.55 90)
-			(effects
-				(font
-					(size 1.27 1.27)
-				)
-			)
-		)
-		(property "Footprint" "Diode_THT:D_DO-41_SOD81_P7.62mm_Horizontal"
-			(at 127 83.82 0)
-			(effects
-				(font
-					(size 1.27 1.27)
-				)
-				(hide yes)
-			)
-		)
-		(property "Datasheet" "~"
-			(at 127 83.82 0)
-			(effects
-				(font
-					(size 1.27 1.27)
-				)
-				(hide yes)
-			)
-		)
-		(property "Description" "Diode"
-			(at 127 83.82 0)
-			(effects
-				(font
-					(size 1.27 1.27)
-				)
-				(hide yes)
-			)
-		)
-		(property "Sim.Device" "D"
-			(at 127 83.82 0)
-			(effects
-				(font
-					(size 1.27 1.27)
-				)
-				(hide yes)
-			)
-		)
-		(property "Sim.Pins" "1=K 2=A"
-			(at 127 83.82 0)
-			(effects
-				(font
-					(size 1.27 1.27)
-				)
-				(hide yes)
-			)
-		)
-		(pin "2"
-		)
-		(pin "1"
-		)
-		(instances
-			(project "NosLed"
-				(path "/473a9690-2801-417b-8084-b7ef486d51ca/62dae79f-20f1-42ce-ac91-8f6732a4f040"
-					(reference "D501")
-					(unit 1)
-				)
+					(reference "R503")
+					(unit 1)
+				)

Commit message: Tracing draft
Parts:
- renumbered C501 to C301, D502 to D301, L501 to L301, R501 to R301, R502 to R302, R503 to R303, U502 to U301
Changed lines of the file:
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@@
 		(on_board yes)
 		(dnp no)
-		(property "Reference" "L501"
+		(property "Reference" "L301"
 			(at 144.526 89.154 90)
 			(effects
@@
 				(path "/473a9690-2801-417b-8084-b7ef486d51ca/62dae79f-20f1-42ce-ac91-8f6732a4f040"
 					(reference "L501")
+					(unit 1)
+				)
+				(path "/473a9690-2801-417b-8084-b7ef486d51ca/cce27811-e524-4674-b3ee-a0b5fcce088d"
+					(reference "L301")
 					(unit 1)
 				)
@@
 		(dnp no)
 		(fields_autoplaced yes)
-		(property "Reference" "U502"
+		(property "Reference" "U301"
 			(at 111.3633 87.63 0)
 			(effects
@@
 				(path "/473a9690-2801-417b-8084-b7ef486d51ca/62dae79f-20f1-42ce-ac91-8f6732a4f040"
 					(reference "U502")
+					(unit 1)
+				)
+				(path "/473a9690-2801-417b-8084-b7ef486d51ca/cce27811-e524-4674-b3ee-a0b5fcce088d"
+					(reference "U301")
 					(unit 1)
 				)
@@
 		(dnp no)
 		(fields_autoplaced yes)
-		(property "Reference" "D502"
+		(property "Reference" "D301"
 			(at 129.54 82.5499 90)
 			(effects
@@
 				(path "/473a9690-2801-417b-8084-b7ef486d51ca/62dae79f-20f1-42ce-ac91-8f6732a4f040"
 					(reference "D502")
+					(unit 1)
+				)
+				(path "/473a9690-2801-417b-8084-b7ef486d51ca/cce27811-e524-4674-b3ee-a0b5fcce088d"
+					(reference "D301")
 					(unit 1)
 				)
@@
 		(dnp no)
 		(fields_autoplaced yes)
-		(property "Reference" "C501"
+		(property "Reference" "C301"
 			(at 143.51 74.0409 0)
 			(effects
@@
 				(path "/473a9690-2801-417b-8084-b7ef486d51ca/62dae79f-20f1-42ce-ac91-8f6732a4f040"
 					(reference "C501")
+					(unit 1)
+				)
+				(path "/473a9690-2801-417b-8084-b7ef486d51ca/cce27811-e524-4674-b3ee-a0b5fcce088d"
+					(reference "C301")
 					(unit 1)
 				)
@@
 		(on_board yes)
 		(dnp no)
-		(property "Reference" "R502"
+		(property "Reference" "R302"
 			(at 132.334 106.934 90)
 			(effects
@@
 				(path "/473a9690-2801-417b-8084-b7ef486d51ca/62dae79f-20f1-42ce-ac91-8f6732a4f040"
 					(reference "R502")
+					(unit 1)
+				)
+				(path "/473a9690-2801-417b-8084-b7ef486d51ca/cce27811-e524-4674-b3ee-a0b5fcce088d"
+					(reference "R302")
 					(unit 1)
 				)
@@
 		(on_board yes)
 		(dnp no)
-		(property "Reference" "R501"
+		(property "Reference" "R301"
 			(at 94.742 94.234 90)
 			(effects
@@
 				(path "/473a9690-2801-417b-8084-b7ef486d51ca/62dae79f-20f1-42ce-ac91-8f6732a4f040"
 					(reference "R501")
+					(unit 1)
+				)
+				(path "/473a9690-2801-417b-8084-b7ef486d51ca/cce27811-e524-4674-b3ee-a0b5fcce088d"
+					(reference "R301")
 					(unit 1)
 				)
@@
 		(on_board yes)
 		(dnp no)
-		(property "Reference" "R503"
+		(property "Reference" "R303"
 			(at 169.926 74.168 90)
 			(effects
@@
 					(unit 1)
 				)
+				(path "/473a9690-2801-417b-8084-b7ef486d51ca/cce27811-e524-4674-b3ee-a0b5fcce088d"
+					(reference "R303")
+					(unit 1)
+				)
