File: hardware/NosLed.kicad_pcb (KiCad board)
At the start: 2 copper layers, 25.4 x 61 mm, 23 parts, among them J101 LOAD, J102 PWM, J201 AC, U101 BP2876, U102 PC817

Commit message: AC Input
Parts:
- removed the C202 at (155.0, 149.9)
- removed F201: Fuse, Fuse:Fuseholder_Cylinder-5x20mm_Stelvio-Kontek_PTF78_Horizontal_Open
- removed J201: AC, TerminalBlock_Phoenix:TerminalBlock_Phoenix_MKDS-1,5-2-5.08_1x02_P5.08mm_Horizontal
- removed NT202: NetTie_2, NetTie:NetTie-2_SMD_Pad0.5mm
- removed R101: 330R, Resistor_THT:R_Axial_DIN0207_L6.3mm_D2.5mm_P7.62mm_Horizontal
- removed R204: 51K, Resistor_THT:R_Axial_DIN0207_L6.3mm_D2.5mm_P7.62mm_Horizontal
- removed U102: PC817, Package_DIP:DIP-4_W7.62mm
- added C201: MKP X2 275VAC, Capacitor_THT:C_Rect_L13.0mm_W6.0mm_P10.00mm_FKS3_FKP3_MKS4, F.Cu at (83.8, 72.4)
- added C203: 22uF 400v, Capacitor_THT:CP_Radial_D13.0mm_P5.00mm, F.Cu at (89.0, 116.8)
- added J101: AC, TerminalBlock_Phoenix:TerminalBlock_Phoenix_MKDS-1,5-2-5.08_1x02_P5.08mm_Horizontal, F.Cu at (83.8, 57.1)
- added J103: 380OUT, TerminalBlock_Phoenix:TerminalBlock_Phoenix_MKDS-1,5-2-5.08_1x02_P5.08mm_Horizontal, F.Cu at (88.9, 128.3)
- added J104: 380OUT, TerminalBlock_Phoenix:TerminalBlock_Phoenix_MKDS-1,5-2-5.08_1x02_P5.08mm_Horizontal, F.Cu at (116.8, 124.5)
- added L201: 1mH 0.5A, Inductor_THT:L_Radial_D10.0mm_P5.00mm_Fastron_07M, F.Cu at (81.3, 106.8)
- added NT303: NetTie_2, NetTie:NetTie-2_SMD_Pad0.5mm, B.Cu at (127.0, 67.3)
- added R201: Fusible 10R 1W, Resistor_THT:R_Axial_DIN0414_L11.9mm_D4.5mm_P15.24mm_Horizontal, F.Cu at (78.7, 57.1)
- added R202: 1M 0.5W, Resistor_THT:R_Axial_DIN0309_L9.0mm_D3.2mm_P12.70mm_Horizontal, F.Cu at (94.0, 77.5)
- C202: renamed from C204; value 33uF 400v -> 22uF 400v
- C302: renamed from C203; value 10uF 63v -> 10uF 100v; footprint Capacitor_THT:CP_Radial_D5.0mm_P2.50mm -> Capacitor_THT:CP_Radial_D6.3mm_P2.50mm
- D201: value MB10S -> MB10M
- NT301: renamed from NT201; moved to B.Cu
- NT302: renamed from NT203; moved to B.Cu
- R301: renamed from R202; footprint Resistor_THT:R_Axial_DIN0207_L6.3mm_D2.5mm_P7.62mm_Horizontal -> Resistor_THT:R_Axial_DIN0309_L9.0mm_D3.2mm_P12.70mm_Horizontal
- R302: renamed from R203; value 10K -> 27K
- moved RV201 97.6 mm to (91.3, 66.8), turned to 180 degrees
- moved D201 71.8 mm to (91.4, 86.4), turned to -90 degrees
- moved NT302 59.7 mm to (117.3, 76.2), turned to 180 degrees
- moved C202 58.6 mm to (89.0, 101.6), turned to 0 degrees
- moved NT301 45.9 mm to (132.1, 95.3)
- moved C302 41.0 mm to (134.7, 111.8)
- moved L301 39.8 mm to (134.7, 101.6)
- moved D301 37.8 mm to (137.2, 91.4), turned to 90 degrees
- moved J102 37.4 mm to (115.6, 66.8), turned to 0 degrees
- moved J105 36.4 mm to (134.6, 124.5)
- moved R304 35.4 mm to (127.0, 66.0)
- moved U301 35.3 mm to (132.1, 71.1)
- moved R302 33.1 mm to (129.5, 76.2)
- moved C301 32.6 mm to (126.9, 81.3)
- moved R301 31.8 mm to (132.1, 81.3), turned to -90 degrees
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- renumbered C201 to C301, D202 to D301, J101 to J105, L201 to L301, R201 to R304, R205 to R305, U101 to U301
Connections:
- net /BP2876/CS renamed /BP2876D/CS
- net /BP2876/DRAIN renamed /BP2876D/DRAIN
- C202 pad 1: /BP2876/LOAD+ -> Net-(D201-+)
- C202 pad 2: /BP2876/PWR_GND -> /BP2876D/PWR_GND
- C301 pad 2: Net-(U101-GND) -> Net-(C301-Pad2)
- C302 pad 1: /BP2876/LOAD+ -> /ACInput/380V
- C302 pad 2: Net-(C202-Pad1) -> /BP2876D/LOAD-
- D201 pad 1: /BP2876/AC_FUSE -> /ACInput/AC_N
- D201 pad 2: /BP2876/AC_L -> /ACInput/AC_L_FUSE
- D201 pad 3: /BP2876/LOAD+ -> Net-(D201-+)
- D201 pad 4: /BP2876/PWR_GND -> /BP2876D/PWR_GND
- D301 pad 1: /BP2876/LOAD+ -> /ACInput/380V
- J102 pad 1: /BP2876/HI_GND -> /BP2876D/PWM
- J102 pad 2: /BP2876/PWM -> /BP2876D/PWR_GND
- J105 pad 1: /BP2876/LOAD+ -> /ACInput/380V
- J105 pad 2: /BP2876/LOAD- -> /BP2876D/LOAD-
- L301 pad 1: /BP2876/LOAD- -> /BP2876D/LOAD-
- NT301 pad 2: /BP2876/LOAD+ -> /ACInput/380V
- NT302 pad 1: /BP2876/PWR_GND -> Net-(C301-Pad2)
- NT302 pad 2: Net-(U101-GND) -> /BP2876D/PWR_GND
- R302 pad 2: Net-(U101-GND) -> Net-(C301-Pad2)
- R304 pad 1: /BP2876/PWR_GND -> /BP2876D/PWR_GND
- R305 pad 1: /BP2876/LOAD+ -> /ACInput/380V
- R305 pad 2: /BP2876/LOAD- -> /BP2876D/LOAD-
- RV201 pad 1: /BP2876/AC_L -> /ACInput/AC_N
- RV201 pad 2: /BP2876/AC_FUSE -> /ACInput/AC_L_FUSE
- U301 pad 1: Net-(U101-GND) -> Net-(U301-GND)
- U301 pad 2: /BP2876/PWM -> /BP2876D/PWM
Routing:
- net /BP2876D/PWR_GND: track 0.00 -> 66.6 mm
- net /ACInput/380V: track 0.00 -> 53.0 mm
- net /BP2876D/DRAIN: track 0.00 -> 31.5 mm
- net /BP2876D/LOAD-: track 0.00 -> 24.9 mm
- net /BP2876D/PWM: track 0.00 -> 19.1 mm
- net Net-(U301-VCC): track 0.00 -> 11.3 mm
- net Net-(C301-Pad2): track 0.00 -> 10.8 mm
- net Net-(U301-GND): track 0.00 -> 6.47 mm
Other:
- board size 25.4 x 61 mm -> 63.5 x 73.7 mm

Commit message: LNK302PN
Parts:
- added C401: 100nF, Capacitor_THT:C_Disc_D5.0mm_W2.5mm_P5.00mm, F.Cu at (88.9, 137.1)
- added C402: 10uF 16V, Capacitor_THT:CP_Radial_D5.0mm_P2.50mm, F.Cu at (99.1, 129.5)
- added C403: 470uF 10V, Capacitor_THT:CP_Radial_D10.0mm_P5.00mm, F.Cu at (116.8, 129.5)
- added C404: 100nF, Capacitor_THT:C_Disc_D5.0mm_W2.5mm_P5.00mm, F.Cu at (124.5, 134.5)
- added C405: 100nF, Capacitor_THT:C_Disc_D5.0mm_W2.5mm_P5.00mm, F.Cu at (139.7, 134.5)
- added C406: 22uF 10V, Capacitor_THT:CP_Radial_D6.3mm_P2.50mm, F.Cu at (134.6, 132.1)
- added D401: ES1J (UF4007), Diode_THT:D_DO-41_SOD81_P7.62mm_Horizontal, F.Cu at (94.0, 132.1)
- added D402: 1N4007, Diode_THT:D_DO-41_SOD81_P7.62mm_Horizontal, F.Cu at (101.6, 127.0)
- added J107: 3V3, TerminalBlock_Phoenix:TerminalBlock_Phoenix_MKDS-1,5-2-5.08_1x02_P5.08mm_Horizontal, F.Cu at (144.8, 129.5)
- added J108: 380_LNK302PN, TerminalBlock_Phoenix:TerminalBlock_Phoenix_MKDS-1,5-2-5.08_1x02_P5.08mm_Horizontal, F.Cu at (73.7, 134.6)
- added L401: 2.2mH, Inductor_THT:L_Radial_D10.0mm_P5.00mm_Fastron_07M, F.Cu at (106.7, 137.2)
- added R401: 2.2K, Resistor_THT:R_Axial_DIN0207_L6.3mm_D2.5mm_P7.62mm_Horizontal, F.Cu at (91.4, 137.2)
- added R402: 4.7K, Resistor_THT:R_Axial_DIN0207_L6.3mm_D2.5mm_P7.62mm_Horizontal, F.Cu at (99.1, 127.0)
- added U401: AMS1117-3.3, Package_TO_SOT_SMD:SOT-223-3_TabPin2, F.Cu at (126.4, 132.3)
- added U402: LNK306P, Package_DIP:PowerIntegrations_PDIP-8B, F.Cu at (86.4, 137.2)
- J104: value 380OUT -> 380_BP2876D
- moved R304 67.1 mm to (73.7, 83.8)
- moved C202 67.1 mm to (30.6, 68.6)
- moved C203 67.1 mm to (30.6, 83.8)
- moved C301 67.1 mm to (68.5, 48.3)
- moved C302 67.1 mm to (76.2, 78.7)
- moved D301 67.1 mm to (78.7, 58.4)
- moved J103 67.1 mm to (30.5, 95.2)
- moved J104 67.1 mm to (58.4, 91.4)
- moved J105 67.1 mm to (76.2, 91.4)
- moved L201 67.1 mm to (22.9, 73.7)
- moved NT301 67.1 mm to (58.9, 43.2)
- moved NT302 67.1 mm to (73.7, 62.3)
- moved NT303 67.1 mm to (68.6, 34.2)
- moved R202 67.1 mm to (35.6, 44.5)
- moved R301 67.1 mm to (73.7, 48.3)
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- renumbered NT302 to NT301, NT301 to NT302, R304 to R303, R305 to R304
Routing:
- net /BP2876D/PWR_GND: track 66.6 -> 150.7 mm
- net Net-(D401-K): track 0.00 -> 46.4 mm
- net /ACInput/AC_L_FUSE: track 0.00 -> 35.5 mm
- net /ACInput/AC_N: track 0.00 -> 32.4 mm
- net /LNK302PN/5V: track 0.00 -> 27.8 mm, vias 0 -> 1
- net Net-(D201-+): track 0.00 -> 17.5 mm
- net /LNK302PN/3V3: track 0.00 -> 16.4 mm, vias 0 -> 1
- net /ACInput/380V: track 53.0 -> 67.8 mm
- net Net-(U402-FB): track 0.00 -> 7.62 mm
- net /ACInput/AC_L: track 0.00 -> 5.08 mm
- net Net-(D402-K): track 0.00 -> 5.08 mm
- net Net-(U402-BP): track 0.00 -> 2.54 mm
- net Net-(U301-ROVP): track 0.00 -> 2.54 mm
Other:
- board size 63.5 x 73.7 mm -> 127 x 118.1 mm

Commit message: BP2956XS
Parts:
- added C502: 10uF 100v, Capacitor_THT:CP_Radial_D6.3mm_P2.50mm, F.Cu at (114.3, 81.3)
- added D501: UF4007, Diode_THT:D_DO-41_SOD81_P7.62mm_Horizontal, F.Cu at (116.8, 55.9)
- added J106: PWM1, TerminalBlock_Phoenix:TerminalBlock_Phoenix_MKDS-1-2-3.81_1x02_P3.81mm_Horizontal, F.Cu at (109.2, 30.5)
- added J109: 380_BP2956XS, TerminalBlock_Phoenix:TerminalBlock_Phoenix_MKDS-1,5-2-5.08_1x02_P5.08mm_Horizontal, F.Cu at (109.2, 53.3)
- added J110: LOAD2, TerminalBlock_Phoenix:TerminalBlock_Phoenix_MKDS-1,5-2-5.08_1x02_P5.08mm_Horizontal, F.Cu at (114.3, 96.5)
- added L501: 2.2mH, Inductor_THT:L_Radial_D10.0mm_P5.00mm_Fastron_07M, F.Cu at (124.5, 68.6)
- added R502: 7K5, Resistor_THT:R_Axial_DIN0207_L6.3mm_D2.5mm_P7.62mm_Horizontal, F.Cu at (119.4, 40.6)
- added R503: 2R7, Resistor_THT:R_Axial_DIN0309_L9.0mm_D3.2mm_P12.70mm_Horizontal, F.Cu at (111.8, 43.2)
- added R504: 100К, Resistor_THT:R_Axial_DIN0207_L6.3mm_D2.5mm_P7.62mm_Horizontal, F.Cu at (114.3, 91.4)
- added U502: BP2956XS, Package_DIP:DIP-8_W7.62mm, F.Cu at (116.8, 45.7)
- C202, C203: value 22uF 400v -> 15uF 400v
- C406: value 22uF 10V -> 100uF 10V
- D401: value ES1J (UF4007) -> ES1J
- D402: value 1N4007 -> US1M
- J102: value PWM -> PWM2
- J105: value LOAD -> LOAD2
Routing:
- net /ACInput/380V: track 67.8 -> 122.2 mm
- net /BP2956XS/LOAD-: track 0.00 -> 34.3 mm
- net /BP2956XS/PWM: track 0.00 -> 24.1 mm
- net /BP2876D/PWR_GND: track 150.7 -> 172.9 mm
- net /BP2956XS/DRAIN: track 0.00 -> 17.3 mm
- net Net-(U502-ROVP): track 0.00 -> 6.13 mm
- net /BP2956XS/CS: track 0.00 -> 2.54 mm
Other:
- outline, holes or cut-outs redrawn

Commit message: Prototype
Parts:
- removed D501: UF4007, Diode_THT:D_DO-41_SOD81_P7.62mm_Horizontal
- removed the J106 at (109.2, 30.5)
- removed J109: 380_BP2956XS, TerminalBlock_Phoenix:TerminalBlock_Phoenix_MKDS-1,5-2-5.08_1x02_P5.08mm_Horizontal
- removed the J110 at (114.3, 96.5)
- added C602: 100nF, Capacitor_THT:C_Disc_D5.0mm_W2.5mm_P5.00mm, F.Cu at (241.3, 93.9)
- added C603: 100uF 10V, Capacitor_THT:CP_Radial_D6.3mm_P2.50mm, F.Cu at (243.8, 88.8)
- added C604: 1uF (2.2uF) 16v (25v), Capacitor_THT:C_Disc_D5.0mm_W2.5mm_P5.00mm, F.Cu at (236.2, 86.4)
- added C605: 100nF, Capacitor_THT:C_Disc_D5.0mm_W2.5mm_P5.00mm, F.Cu at (248.9, 83.7)
- added C606: 330uF (470uF) 16v, Capacitor_THT:CP_Radial_D6.3mm_P2.50mm, F.Cu at (226.0, 104.1)
- added D502: US1M, Diode_SMD:D_SMA, F.Cu at (22.0, 38.0)
- added J112: LOAD2, TerminalBlock_Phoenix:TerminalBlock_Phoenix_MKDS-1,5-2-5.08_1x02_P5.08mm_Horizontal, F.Cu at (254.0, 88.8)
- added L601: 680uH (1mH), Inductor_THT:L_Radial_D10.0mm_P5.00mm_Fastron_07M, F.Cu at (233.7, 99.1)
- added TP101: TestPoint, TestPoint:TestPoint_Pad_4.0x4.0mm, F.Cu at (22.5, 17.0)
- added TP102: TestPoint, TestPoint:TestPoint_Pad_4.0x4.0mm, F.Cu at (16.0, 17.0)
- added TP103: TestPoint, TestPoint:TestPoint_Pad_4.0x4.0mm, F.Cu at (19.0, 78.0)
- added TP104: TestPoint, TestPoint:TestPoint_Pad_4.0x4.0mm, F.Cu at (26.0, 78.0)
- added TP105: TestPoint, TestPoint:TestPoint_Pad_4.0x4.0mm, F.Cu at (29.0, 24.0)
- added TP106: TestPoint, TestPoint:TestPoint_Pad_4.0x4.0mm, F.Cu at (29.0, 17.0)
- added U601: BP8501CH, Package_DIP:DIP-8_W7.62mm, F.Cu at (226.1, 86.3)
- added U602: AMS1117-3.3, Package_TO_SOT_SMD:SOT-223-3_TabPin2, F.Cu at (247.0, 96.2)
- C501: renamed from C502; footprint Capacitor_THT:CP_Radial_D6.3mm_P2.50mm -> Capacitor_THT:CP_Radial_D10.0mm_P5.00mm
- R501: renamed from R502; footprint Resistor_THT:R_Axial_DIN0207_L6.3mm_D2.5mm_P7.62mm_Horizontal -> Resistor_SMD:R_0805_2012Metric_Pad1.20x1.40mm_HandSolder
- R502: renamed from R503; footprint Resistor_THT:R_Axial_DIN0309_L9.0mm_D3.2mm_P12.70mm_Horizontal -> Resistor_SMD:R_1206_3216Metric_Pad1.30x1.75mm_HandSolder
- R503: renamed from R504; footprint Resistor_THT:R_Axial_DIN0207_L6.3mm_D2.5mm_P7.62mm_Horizontal -> Resistor_SMD:R_1206_3216Metric_Pad1.30x1.75mm_HandSolder
- U502: footprint Package_DIP:DIP-8_W7.62mm -> Package_SO:SOIC-8_5.3x5.3mm_P1.27mm
- moved J102 215.5 mm to (271.9, 50.2), turned to 0 degrees
- moved U401 197.5 mm to (269.4, 62.9), turned to 90 degrees
- moved C402 194.3 mm to (269.5, 65.4), turned to 0 degrees
- moved R401 190.9 mm to (269.4, 68.0), turned to 0 degrees
- moved D401 190.7 mm to (274.5, 70.5), turned to 180 degrees
- moved R402 187.7 mm to (279.5, 75.6), turned to 90 degrees
- moved C404 185.9 mm to (277.0, 75.6), turned to 180 degrees
- moved D402 184.5 mm to (279.5, 78.1), turned to -90 degrees
- moved L401 171.4 mm to (269.4, 83.2), turned to 0 degrees
- moved C406 164.2 mm to (277.0, 93.4), turned to 180 degrees
- moved C401 151.3 mm to (272.0, 101.0), turned to 0 degrees
- moved U402 150.7 mm to (274.2, 102.9), turned to 90 degrees
- moved C403 141.4 mm to (274.4, 111.2), turned to 180 degrees
- moved C405 133.6 mm to (272.0, 116.2), turned to 0 degrees
- moved J108 132.5 mm to (277.0, 121.3), turned to 180 degrees
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- renumbered C404 to C401, C401 to C402, C406 to C403, C402 to C404, C403 to C406, J108 to J102, J102 to J105, J104 to J106, J107 to J108, J105 to J110, U402 to U401, U401 to U402
Connections:
- net /ACInput/380V renamed /ACInput/325V
Routing:
- net /BP2956XS/PWM: track 24.1 -> 7.84 mm
- net /ACInput/325V: track 122.2 -> 135.5 mm
- net /BP2876D/PWR_GND: track 172.9 -> 175.7 mm
- net /BP2956XS/LOAD-: track 34.3 -> 31.6 mm
- net /BP2956XS/CS: track 2.54 -> 5.18 mm
- net Net-(U502-ROVP): track 6.13 -> 3.60 mm
- net /BP2956XS/DRAIN: track 17.3 -> 18.8 mm
Other:
- board size 127 x 118.1 mm -> 150.2 x 99.7 mm

Commit message: Tracing draft
Parts:
- removed C203: 15uF 400v, Capacitor_THT:CP_Radial_D13.0mm_P5.00mm
- removed C404: 10uF 16V, Capacitor_THT:CP_Radial_D5.0mm_P2.50mm
- removed C405, C602, C605: 100nF, Capacitor_THT:C_Disc_D5.0mm_W2.5mm_P5.00mm
- removed C406: 470uF 10V, Capacitor_THT:CP_Radial_D10.0mm_P5.00mm
- removed C603: 100uF 10V, Capacitor_THT:CP_Radial_D6.3mm_P2.50mm
- removed C604: 1uF (2.2uF) 16v (25v), Capacitor_THT:C_Disc_D5.0mm_W2.5mm_P5.00mm
- removed C606: 330uF (470uF) 16v, Capacitor_THT:CP_Radial_D6.3mm_P2.50mm
- removed D502: US1M, Diode_SMD:D_SMA
- removed J105: PWM2, TerminalBlock_Phoenix:TerminalBlock_Phoenix_MKDS-1-2-3.81_1x02_P3.81mm_Horizontal
- removed J106: 380_BP2876D, TerminalBlock_Phoenix:TerminalBlock_Phoenix_MKDS-1,5-2-5.08_1x02_P5.08mm_Horizontal
- removed J108: 3V3, TerminalBlock_Phoenix:TerminalBlock_Phoenix_MKDS-1,5-2-5.08_1x02_P5.08mm_Horizontal
- removed J110, J112: LOAD2, TerminalBlock_Phoenix:TerminalBlock_Phoenix_MKDS-1,5-2-5.08_1x02_P5.08mm_Horizontal
- removed L201: 1mH 0.5A, Inductor_THT:L_Radial_D10.0mm_P5.00mm_Fastron_07M
- removed L601: 680uH (1mH), Inductor_THT:L_Radial_D10.0mm_P5.00mm_Fastron_07M
- removed NT301, NT302, NT303: NetTie_2, NetTie:NetTie-2_SMD_Pad0.5mm
- removed TP101, TP102, TP103, TP104, TP105, TP106: TestPoint, TestPoint:TestPoint_Pad_4.0x4.0mm
- removed U402, U602: AMS1117-3.3, Package_TO_SOT_SMD:SOT-223-3_TabPin2
- removed U502: BP2956XS, Package_SO:SOIC-8_5.3x5.3mm_P1.27mm
- removed U601: BP8501CH, Package_DIP:DIP-8_W7.62mm
- added C101: 1uF, Capacitor_SMD:C_0805_2012Metric_Pad1.18x1.45mm_HandSolder, F.Cu at (59.7, 80.4)
- added C102: 100nF, Capacitor_SMD:C_0805_2012Metric_Pad1.18x1.45mm_HandSolder, F.Cu at (58.0, 92.8)
- added C103: 100uF 10V, Capacitor_THT:CP_Radial_D6.3mm_P2.50mm, F.Cu at (51.3, 81.8)
- added C104: 100nF, Capacitor_SMD:C_0805_2012Metric_Pad1.18x1.45mm_HandSolder, F.Cu at (48.2, 77.2)
- added C502: 10uF 100v, Capacitor_THT:CP_Radial_D6.3mm_P2.50mm, F.Cu at (34.4, 126.3)
- added D501: US1M, Diode_SMD:D_SMA, F.Cu at (32.8, 119.3)
- added G***: LOGO, LOGO, F.Cu at (22.4, 73.3)
- added H101: MountingHole, MountingHole:MountingHole_3.2mm_M3_Pad_Via, F.Cu at (62.5, 135.6)
- added H102: MountingHole, MountingHole:MountingHole_3.2mm_M3_Pad_Via, F.Cu at (34.5, 135.6)
- added H103: MountingHole, MountingHole:MountingHole_3.2mm_M3_Pad_Via, F.Cu at (34.5, 42.5)
- added H104: MountingHole, MountingHole:MountingHole_3.2mm_M3_Pad_Via, F.Cu at (62.5, 42.5)
- added R101: 10K, Resistor_SMD:R_0603_1608Metric_Pad0.98x0.95mm_HandSolder, F.Cu at (63.9, 80.4)
- added R102: 10K, Resistor_SMD:R_0603_1608Metric_Pad0.98x0.95mm_HandSolder, F.Cu at (55.4, 80.4)
- added R103: 5.1K, Resistor_SMD:R_0603_1608Metric_Pad0.98x0.95mm_HandSolder, F.Cu at (54.6, 54.9)
- added R104: 5.1K, Resistor_SMD:R_0603_1608Metric_Pad0.98x0.95mm_HandSolder, F.Cu at (55.2, 48.9)
- added R105: 4.7K, Resistor_SMD:R_0603_1608Metric_Pad0.98x0.95mm_HandSolder, F.Cu at (46.0, 113.0)
- added R106: 4.7K, Resistor_SMD:R_0603_1608Metric_Pad0.98x0.95mm_HandSolder, F.Cu at (64.3, 113.0)
- added R504: 100К, Resistor_SMD:R_1206_3216Metric_Pad1.30x1.75mm_HandSolder, F.Cu at (39.0, 130.7)
- added TP_101: BOOT, NosLib:TestPoint_Pad_1.0x1.0mm, F.Cu at (63.0, 93.9)
- added TP_102: GND, NosLib:TestPoint_Pad_1.0x1.0mm, F.Cu at (63.0, 97.0)
- added TP_103: EN, NosLib:TestPoint_Pad_1.0x1.0mm, F.Cu at (62.9, 99.8)
- added U101: AMS1117-3.3, Package_TO_SOT_SMD:SOT-223-3_TabPin2, F.Cu at (58.3, 86.4)
- added U102: ESP32-C3-WROOM-02U, RF_Module:ESP32-C3-WROOM-02U, F.Cu at (58.9, 68.3)
- added U501: BP2876, Package_SO:SOIC-8-N7_3.9x4.9mm_P1.27mm, F.Cu at (43.9, 108.5)
- C202: value 15uF 400v -> 22uF 400v; footprint Capacitor_THT:CP_Radial_D13.0mm_P5.00mm -> Capacitor_THT:CP_Radial_D10.0mm_P5.00mm
- C301: footprint Capacitor_THT:C_Disc_D5.0mm_W2.5mm_P5.00mm -> Capacitor_SMD:C_0805_2012Metric_Pad1.18x1.45mm_HandSolder
- C401: footprint Capacitor_THT:C_Disc_D5.0mm_W2.5mm_P5.00mm -> Capacitor_SMD:C_0201_0603Metric_Pad0.64x0.40mm_HandSolder
- C402: value 100nF -> 10uF 16V; footprint Capacitor_THT:C_Disc_D5.0mm_W2.5mm_P5.00mm -> Capacitor_SMD:C_0805_2012Metric_Pad1.18x1.45mm_HandSolder
- C403: value 100uF 10V -> 470uF 10V; footprint Capacitor_THT:CP_Radial_D6.3mm_P2.50mm -> Capacitor_THT:CP_Radial_D10.0mm_P5.00mm
- C501: value 10uF 100v -> 4.7uF 25v; footprint Capacitor_THT:CP_Radial_D10.0mm_P5.00mm -> Capacitor_SMD:C_0805_2012Metric_Pad1.18x1.45mm_HandSolder
- D201: value MB10M -> MB10S; footprint Package_DIP:DIP-4_W7.62mm -> Package_TO_SOT_SMD:TO-269AA
- D301: value UF4007 -> US1M; footprint Diode_THT:D_DO-41_SOD81_P7.62mm_Horizontal -> Diode_SMD:D_SMA
- D401: value ES1J -> US1M; footprint Diode_THT:D_DO-41_SOD81_P7.62mm_Horizontal -> Diode_SMD:D_SMA
- D402: footprint Diode_THT:D_DO-41_SOD81_P7.62mm_Horizontal -> Diode_SMD:D_SMA
- J102: value 380_LNK302PN -> USB_C_Receptacle_USB2.0_16P; footprint TerminalBlock_Phoenix:TerminalBlock_Phoenix_MKDS-1,5-2-5.08_1x02_P5.08mm_Horizontal -> Connector_USB:USB_C_Receptacle_HRO_TYPE-C-31-M-12
- J103: value 380OUT -> LOAD; footprint TerminalBlock_Phoenix:TerminalBlock_Phoenix_MKDS-1,5-2-5.08_1x02_P5.08mm_Horizontal -> TerminalBlock_Phoenix:TerminalBlock_Phoenix_MKDS-1,5-3-5.08_1x03_P5.08mm_Horizontal
- L301, L401, L501: footprint Inductor_THT:L_Radial_D10.0mm_P5.00mm_Fastron_07M -> Inductor_THT:L_Radial_D12.0mm_P5.00mm_Neosid_SD12k_style2
- R202: footprint Resistor_THT:R_Axial_DIN0309_L9.0mm_D3.2mm_P12.70mm_Horizontal -> Resistor_SMD:R_2512_6332Metric_Pad1.40x3.35mm_HandSolder
- R301: value 680K -> 470K; footprint Resistor_THT:R_Axial_DIN0309_L9.0mm_D3.2mm_P12.70mm_Horizontal -> Resistor_SMD:R_2512_6332Metric_Pad1.40x3.35mm_HandSolder
- R302: value 27K -> 22K; footprint Resistor_THT:R_Axial_DIN0207_L6.3mm_D2.5mm_P7.62mm_Horizontal -> Resistor_SMD:R_0201_0603Metric_Pad0.64x0.40mm_HandSolder
- R303: value 3R3 -> 2.7; footprint Resistor_THT:R_Axial_DIN0309_L9.0mm_D3.2mm_P12.70mm_Horizontal -> Resistor_SMD:R_0805_2012Metric_Pad1.20x1.40mm_HandSolder
- R304: footprint Resistor_THT:R_Axial_DIN0207_L6.3mm_D2.5mm_P7.62mm_Horizontal -> Resistor_SMD:R_1206_3216Metric_Pad1.30x1.75mm_HandSolder
- R401, R402: footprint Resistor_THT:R_Axial_DIN0207_L6.3mm_D2.5mm_P7.62mm_Horizontal -> Resistor_SMD:R_0201_0603Metric_Pad0.64x0.40mm_HandSolder
- R501: value 7K5 -> 470K; footprint Resistor_SMD:R_0805_2012Metric_Pad1.20x1.40mm_HandSolder -> Resistor_SMD:R_2512_6332Metric_Pad1.40x3.35mm_HandSolder
- R502: value 2R7 -> 22K; footprint Resistor_SMD:R_1206_3216Metric_Pad1.30x1.75mm_HandSolder -> Resistor_SMD:R_0201_0603Metric_Pad0.64x0.40mm_HandSolder
- R503: value 100К -> 2.7; footprint Resistor_SMD:R_1206_3216Metric_Pad1.30x1.75mm_HandSolder -> Resistor_SMD:R_0805_2012Metric_Pad1.20x1.40mm_HandSolder
- U301: footprint Package_DIP:DIP-8-N7_W7.62mm -> Package_SO:SOIC-8-N7_3.9x4.9mm_P1.27mm
- U401: value LNK306P -> LNK306D; footprint Package_DIP:PowerIntegrations_PDIP-8B -> Package_SO:SOIC-8_3.9x4.9mm_P1.27mm
- moved D402 245.8 mm to (34.9, 102.5), turned to 180 degrees
- moved R402 242.2 mm to (38.0, 93.4), turned to 180 degrees
- moved C402 238.1 mm to (33.7, 98.4), turned to 180 degrees
- moved U401 237.6 mm to (33.7, 92.9), turned to -90 degrees
- moved C401 234.3 mm to (38.0, 89.8), turned to 180 degrees
- moved R401 232.7 mm to (37.9, 91.6), turned to 180 degrees
- moved D401 232.7 mm to (43.9, 101.8), turned to 0 degrees
- moved L401 223.8 mm to (45.8, 94.1), turned to 90 degrees
- moved C403 218.2 mm to (56.5, 99.9)
- moved J102 210.1 mm to (61.8, 51.3), turned to 90 degrees
- moved R301 147.3 mm to (51.3, 109.7)
- moved R303 144.9 mm to (55.9, 107.5), turned to 90 degrees
- moved L301 143.4 mm to (55.3, 123.3), turned to 90 degrees
- moved R302 141.8 mm to (59.4, 113.3), turned to 0 degrees
- moved U301 141.7 mm to (62.3, 108.5)
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Connections:
- net /BP2876D/CS renamed /BP2876D_WARM/CS
- net /BP2876D/DRAIN renamed /BP2876D_WARM/DRAIN
- C201 pad 2: /ACInput/AC_N -> /ACInput/AC_L
- C202 pad 1: Net-(D201-+) -> /ACInput/325V
- C202 pad 2: /BP2876D/PWR_GND -> GND
- C301 pad 2: Net-(C301-Pad2) -> GND
- C302 pad 2: /BP2876D/LOAD- -> /BP2876D_WARM/LOAD-
- C401 pad 1: /BP2876D/PWR_GND -> Net-(D401-K)
- C401 pad 2: /LNK302PN/5V -> Net-(U401-BP)
- C402 pad 2: Net-(U401-BP) -> Net-(D402-A)
- C403 pad 1: /LNK302PN/3V3 -> 5V
- C403 pad 2: /BP2876D/PWR_GND -> GND
- C501 pad 1: /ACInput/325V -> Net-(U501-VCC)
- C501 pad 2: /BP2956XS/LOAD- -> GND
- D201 pad 1: /ACInput/AC_N -> /ACInput/AC_L
- D201 pad 3: Net-(D201-+) -> /ACInput/325V
- D201 pad 4: /BP2876D/PWR_GND -> GND
- D401 pad 2: /BP2876D/PWR_GND -> GND
- D402 pad 1: Net-(D402-K) -> 5V
- D402 pad 2: /LNK302PN/5V -> Net-(D402-A)
- J103 pad 1: /ACInput/325V -> /BP2876D_COLD/LOAD-
- J103 pad 2: /BP2876D/PWR_GND -> /ACInput/325V
- L301 pad 1: /BP2876D/LOAD- -> /BP2876D_WARM/LOAD-
- L401 pad 2: /LNK302PN/5V -> 5V
- L501 pad 1: /BP2956XS/LOAD- -> /BP2876D_COLD/LOAD-
- L501 pad 2: /BP2956XS/DRAIN -> /BP2876D_COLD/DRAIN
- R201 pad 1: /ACInput/AC_L -> /ACInput/AC_N
- R202 pad 1: /ACInput/AC_N -> /ACInput/AC_L
- R301 pad 2: Net-(NT302-Pad1) -> /ACInput/325V
- R302 pad 2: Net-(C301-Pad2) -> GND
- R303 pad 1: /BP2876D/PWR_GND -> GND
- R304 pad 2: /BP2876D/LOAD- -> /BP2876D_WARM/LOAD-
- R402 pad 1: Net-(D402-K) -> Net-(D402-A)
- R501 pad 1: Net-(U502-ROVP) -> Net-(U501-VCC)
- R501 pad 2: /BP2876D/PWR_GND -> /ACInput/325V
- R502 pad 1: /BP2876D/PWR_GND -> Net-(U501-ROVP)
- R502 pad 2: /BP2956XS/CS -> GND
- R503 pad 1: /ACInput/325V -> GND
- R503 pad 2: /BP2956XS/LOAD- -> /BP2876D_COLD/CS
- RV201 pad 1: /ACInput/AC_N -> /ACInput/AC_L
- U301 pad 1: Net-(U301-GND) -> GND
- U301 pad 2: /BP2876D/PWM -> PWM_WARM
- U401 pad 1: Net-(D401-K) -> Net-(U401-BP)
- U401 pad 2: Net-(D401-K) -> Net-(U401-FB)
- U401 pad 3: Net-(U401-BP) -> (no net)
- U401 pad 4: Net-(U401-FB) -> /ACInput/325V
- U401 pad 5: /ACInput/325V -> Net-(D401-K)
Routing:
- net /BP2876D/PWR_GND: track 175.7 -> 0.00 mm
- net 5V: track 0.00 -> 127.1 mm, vias 0 -> 1
- net GND: track 0.00 -> 61.7 mm
- net PWM_COLD: track 0.00 -> 51.5 mm, vias 0 -> 2
- net PWM_WARM: track 0.00 -> 44.7 mm, vias 0 -> 2
- net /ACInput/325V: track 135.5 -> 94.4 mm, vias 0 -> 2
- net /BP2956XS/LOAD-: track 31.6 -> 0.00 mm
- net /ACInput/AC_L: track 5.08 -> 35.4 mm
- net /LNK302PN/5V: track 27.8 -> 0.00 mm, vias 1 -> 0
- net 3V3: track 0.00 -> 25.7 mm
- net /BP2876D/LOAD-: track 24.9 -> 0.00 mm
- net /BP2876D_COLD/DRAIN: track 0.00 -> 22.9 mm
- net /BP2876D_COLD/LOAD-: track 0.00 -> 20.8 mm
- net /BP2876D_WARM/LOAD-: track 0.00 -> 20.8 mm
- net /ACInput/AC_N: track 32.4 -> 13.1 mm
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- added copper zone on B.Cu, net GND
- added copper zone on F.Cu, net GND
Other:
- board size 150.2 x 99.7 mm -> 37 x 100 mm
