File: hardware/NosLed.kicad_pcb (KiCad board)
At the start: 2 copper layers, 35 x 100 mm, 65 parts, among them J101 USB_C_Receptacle_USB2.0_16P, J102 LOAD, J103 AC, U101 AMS1117-3.3, U102 ESP32-C3-WROOM-02U, U301 BP2876, U401 LNK306D, U501 BP2876

Commit message: v1.1
Parts:
- C102: value 100uF 10V -> 220uF 25V
- C403: value 470uF 10V -> 470uF 16V
- L401: value 2.2mH -> 470uF
- R304, R504: value 2.7 -> 2R7
- U401: footprint Package_SO:SOIC-8_3.9x4.9mm_P1.27mm -> NosLib:LNK302PN-SOIC-8_3.9x4.9mm_P1.27mm
- turned D401 to 90 degrees
Connections:
- C401 pad 2: Net-(D401-A) -> Net-(D401-K)
- D401 pad 1: 5V -> Net-(D401-K)
- D401 pad 2: Net-(D401-A) -> 5V
- R401 pad 1: Net-(D401-A) -> Net-(D401-K)
Routing:
- net Net-(D401-K): track 0.00 -> 5.61 mm
- net Net-(D401-A): track 5.61 -> 0.00 mm
- net Net-(U501-ROVP): track 8.44 -> 10.7 mm
Other:
- board text added: "v1.1"
- board text removed: "v1"
Changed lines of the file:
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@@
 	(net 36 "/LNK302PN/SOURCE")
 	(net 37 "PWR_GND")
-	(net 38 "Net-(D401-A)")
+	(net 38 "Net-(D401-K)")
 	(net 39 "Net-(J101-VBUS-PadA4)")
 	(net 40 "unconnected-(J101-SBU2-PadB8)")
@@
 		(tags "resistor")
 		(property "Reference" "R202"
-			(at 0 -2.63 180)
+			(at 0 2.492811 180)
 			(layer "F.SilkS")
 			(effects
@@
 		(tags "resistor")
 		(property "Reference" "R304"
-			(at 0 -1.65 270)
+			(at 0 1.518652 270)
 			(layer "F.SilkS")
 			(effects
@@
 			)
 		)
-		(property "Value" "2.7"
+		(property "Value" "2R7"
 			(at 0 1.65 270)
 			(layer "F.Fab")
@@
 	(footprint "Diode_SMD:D_SMA"
 		(layer "F.Cu")
-		(at 44.492732 91.10606 -90)
+		(at 44.492732 91.10606 90)
 		(descr "Diode SMA (DO-214AC)")
 		(tags "Diode SMA (DO-214AC)")
 		(property "Reference" "D401"
-			(at -4.434589 0 180)
+			(at 4.357762 0 0)
 			(layer "F.SilkS")
 			(effects
@@
 		)
 		(property "Datasheet" "https://www.diodes.com/assets/Datasheets/ds16008.pdf"
-			(at 0 0 270)
+			(at 0 0 90)
 			(unlocked yes)
 			(layer "F.Fab")
@@
 		)
 		(property "Description" "1000V, 1A, General Purpose Rectifier Diode, SMA(DO-214AC)"
-			(at 0 0 270)
+			(at 0 0 90)
 			(unlocked yes)
 			(layer "F.Fab")
@@
 		)
 		(property "Sim.Device" "D"
-			(at 0 0 270)
+			(at 0 0 90)
 			(unlocked yes)
 			(layer "F.Fab")
@@
 		)
 		(property "Sim.Pins" "1=K 2=A"
-			(at 0 0 270)
+			(at 0 0 90)
 			(unlocked yes)
 			(layer "F.Fab")
@@
 		(attr smd)
 		(fp_line
-			(start -3.51 1.65)
-			(end 2 1.65)
+			(start -3.51 -1.65)
+			(end 2 -1.65)
 			(stroke
 				(width 0.12)
@@
 		)
 		(fp_line
-			(start -3.51 -1.65)
-			(end 2 -1.65)
+			(start -3.51 1.65)
+			(end 2 1.65)
 			(stroke
 				(width 0.12)
@@
 		)
 		(fp_line
-			(start -3.5 1.75)
-			(end -3.5 -1.75)
+			(start 3.5 -1.75)
+			(end 3.5 1.75)
 			(stroke
 				(width 0.05)
@@
 		)
 		(fp_line
-			(start 3.5 1.75)
-			(end -3.5 1.75)
+			(start -3.5 -1.75)
+			(end 3.5 -1.75)
 			(stroke
 				(width 0.05)
@@
 		)
 		(fp_line
-			(start -3.5 -1.75)
-			(end 3.5 -1.75)
+			(start 3.5 1.75)
+			(end -3.5 1.75)
 			(stroke
 				(width 0.05)
@@
 		)
 		(fp_line
-			(start 3.5 -1.75)
-			(end 3.5 1.75)
+			(start -3.5 1.75)
+			(end -3.5 -1.75)
 			(stroke
 				(width 0.05)
@@
 		)
 		(fp_line
-			(start -2.3 1.5)
+			(start 2.3 -1.5)
 			(end -2.3 -1.5)
 			(stroke
@@
 		)
 		(fp_line
-			(start 2.3 1.5)
-			(end -2.3 1.5)
+			(start 2.3 -1.5)
+			(end 2.3 1.5)
 			(stroke
 				(width 0.1)
@@
 		)
 		(fp_line
-			(start 0.50118 0.75032)
-			(end 0.50118 -0.79908)
+			(start -0.64944 -0.79908)
+			(end -0.64944 0.80112)
 			(stroke
 				(width 0.1)
@@
 		)
 		(fp_line
-			(start -0.64944 0.00102)
-			(end 0.50118 0.75032)
+			(start 0.50118 0.00102)
+			(end 1.4994 0.00102)
 			(stroke
 				(width 0.1)
@@
 		(fp_line
 			(start -0.64944 0.00102)
-			(end -1.55114 0.00102)
+			(end 0.50118 -0.79908)
 			(stroke
 				(width 0.1)
@@
 		(fp_line
 			(start -0.64944 0.00102)
-			(end 0.50118 -0.79908)
+			(end -1.55114 0.00102)
 			(stroke
 				(width 0.1)
@@
 		)
 		(fp_line
-			(start 0.50118 0.00102)
-			(end 1.4994 0.00102)
+			(start -0.64944 0.00102)
+			(end 0.50118 0.75032)
 			(stroke
 				(width 0.1)
@@
 		)
 		(fp_line
-			(start -0.64944 -0.79908)
-			(end -0.64944 0.80112)
+			(start 0.50118 0.75032)
+			(end 0.50118 -0.79908)
 			(stroke
 				(width 0.1)
@@
 		)
 		(fp_line
-			(start 2.3 -1.5)
-			(end 2.3 1.5)
+			(start 2.3 1.5)
+			(end -2.3 1.5)
 			(stroke
 				(width 0.1)
@@
 		)
 		(fp_line
-			(start 2.3 -1.5)
+			(start -2.3 1.5)
 			(end -2.3 -1.5)
 			(stroke
@@
 		)
 		(pad "1" smd roundrect
-			(at -2 0 270)
+			(at -2 0 90)
 			(size 2.5 1.8)
 			(layers "F.Cu" "F.Mask" "F.Paste")
 			(roundrect_rratio 0.1388888889)
-			(net 6 "5V")
+			(net 38 "Net-(D401-K)")
 			(pinfunction "K")
 			(pintype "passive")
 		)
 		(pad "2" smd roundrect
-			(at 2 0 270)
+			(at 2 0 90)
 			(size 2.5 1.8)
 			(layers "F.Cu" "F.Mask" "F.Paste")
 			(roundrect_rratio 0.1388888889)
-			(net 38 "Net-(D401-A)")
+			(net 6 "5V")
 			(pinfunction "A")
 			(pintype "passive")
@@
 			(layers "F.Cu" "F.Mask" "F.Paste")
 			(roundrect_rratio 0.25)
-			(net 38 "Net-(D401-A)")
+			(net 38 "Net-(D401-K)")
 			(pintype "passive")
 		)
@@
 		(tags "resistor")
 		(property "Reference" "R106"
-			(at 0 -1.43 180)
+			(at 0 1.557223 180)
 			(layer "F.SilkS")
 			(effects
@@
 		(tags "resistor")
 		(property "Reference" "R501"
-			(at 0 -1.83 180)
+			(at 0 1.932374 180)
 			(layer "F.SilkS")
 			(effects
@@
 			)
 		)
-		(property "Value" "2.2mH"
+		(property "Value" "470uF"
 			(at 2.5 6 90)
 			(layer "F.Fab")
@@
 		)
 	)
-	(footprint "Package_SO:SOIC-8_3.9x4.9mm_P1.27mm"
+	(footprint "NosLib:LNK302PN-SOIC-8_3.9x4.9mm_P1.27mm"
 		(layer "F.Cu")
 		(at 36.536815 101)
@@
 		(tags "SOIC SO")
 		(property "Reference" "U401"
-			(at -4.38581 0.309682 90)
+			(at 0 -3.4 0)
 			(layer "F.SilkS")
 			(effects
@@
 			(pintype "input")
 		)
-		(pad "3" smd roundrect
-			(at -2.475 0.635)
-			(size 1.95 0.6)
-			(layers "F.Cu" "F.Mask" "F.Paste")
-			(roundrect_rratio 0.25)
-		)
 		(pad "4" smd roundrect
 			(at -2.475 1.905)
@@
 		(tags "resistor")
 		(property "Reference" "R302"
-			(at 0 -2.63 270)
+			(at 0.342443 2.580235 270)
 			(layer "F.SilkS")
 			(effects
@@
 		(tags "resistor")
 		(property "Reference" "R502"
-			(at 0 -2.63 270)
+			(at 0 2.741715 270)
 			(layer "F.SilkS")
 			(effects
@@
 		(tags "resistor")
 		(property "Reference" "R504"
-			(at 0 -1.65 270)
+			(at 0 1.615074 270)
 			(layer "F.SilkS")
 			(effects
@@
 			)
 		)
-		(property "Value" "2.7"
+		(property "Value" "2R7"
 			(at 0 1.65 270)
 			(layer "F.Fab")
@@
 			)
 		)
-		(property "Value" "470uF 10V"
+		(property "Value" "470uF 16V"
 			(at 2.5 5.25 90)
 			(layer "F.Fab")
@@
 		(tags "capacitor")
 		(property "Reference" "C302"
-			(at 0 -1.68 90)
+			(at -0.079809 -1.548652 90)
 			(layer "F.SilkS")
 			(effects
@@
 		(tags "TO-269AA MBS diode bridge")
 		(property "Reference" "D201"
-			(at 0 3.374723 180)
+			(at 0.201856 3.374723 180)
 			(layer "F.SilkS")
 			(effects
@@
 		(tags "resistor")
 		(property "Reference" "R401"
-			(at 0 -1.43 180)
+			(at -0.522203 1.413034 180)
 			(layer "F.SilkS")
 			(effects
@@
 			(layers "F.Cu" "F.Mask" "F.Paste")
 			(roundrect_rratio 0.25)
-			(net 38 "Net-(D401-A)")
+			(net 38 "Net-(D401-K)")
 			(pintype "passive")
 		)
@@
 			)
 		)
-		(property "Value" "100uF 10V"
+		(property "Value" "220uF 25V"
 			(at 1.25 4.4 0)
 			(layer "F.Fab")
@@
 		)
 	)
-	(gr_text "v1"
-		(at 62.684376 103.720238 0)
+	(gr_text "v1.1"
+		(at 62.128232 103.678058 0)
 		(layer "F.SilkS")
 		(effects
 			(font
-				(size 1.524 1.524)
-				(thickness 0.3048)
+				(size 1 1)
+				(thickness 0.25)
 				(bold yes)
 			)
@@
 	)
 	(segment
-		(start 43.14 112.320855)
-		(end 43.8 111.660855)
+		(start 41.082022 106.15574)
+		(end 41.835175 106.15574)
 		(width 0.22)
 		(layer "F.Cu")
@@
 	)
 	(segment
-		(start 42.127675 112.320855)
-		(end 43.14 112.320855)
+		(start 43.14 112.320855)
+		(end 43.8 111.660855)
 		(width 0.22)
 		(layer "F.Cu")
@@
 	)
 	(segment
-		(start 42.127654 106.15574)
-		(end 42.847655 106.875741)
+		(start 42.127675 112.320855)
+		(end 43.14 112.320855)
 		(width 0.22)
 		(layer "F.Cu")
@@
 	)
 	(segment
-		(start 41.835175 106.15574)
-		(end 42.127654 106.15574)
+		(start 40.725758 106.512004)
+		(end 41.082022 106.15574)
 		(width 0.22)
 		(layer "F.Cu")
@@
 	)
 	(via
-		(at 42.847655 106.875741)
+		(at 40.725758 106.512004)
 		(size 0.6)
 		(drill 0.3)
@@
 	)
 	(segment
-		(start 42.847655 106.875741)
-		(end 43.8 107.828086)
+		(start 40.725758 106.512004)
+		(end 41.202564 106.98881)
+		(width 0.22)
+		(layer "B.Cu")
+		(net 22)
+	)
+	(segment
+		(start 41.202564 106.98881)
+		(end 42.960724 106.98881)
 		(width 0.22)
 		(layer "B.Cu")
@@
 		(width 0.22)
 		(layer "B.Cu")
+		(net 22)
+	)
+	(segment
+		(start 42.960724 106.98881)
+		(end 43.8 107.828086)
+		(width 0.22)
+		(layer "B.Cu")
