File: hardware/LNK302PN.kicad_sch (KiCad schematic)
At the start: 9 parts, among them U401 LNK306D

Commit message: v1.1
Parts:
- C403: value 470uF 10V -> 470uF 16V
- L401: value 2.2mH -> 470uF
- U401: footprint Package_SO:SOIC-8_3.9x4.9mm_P1.27mm -> NosLib:LNK302PN-SOIC-8_3.9x4.9mm_P1.27mm
Connections:
- net 5V: now also D401.2 (A); no longer D401.1 (K)
- net at C401.2, R401.1: now also D401.1 (K); no longer D401.2 (A)
Changed lines of the file:
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@@
 			)
 		)
-		(property "Value" "470uF 10V"
+		(property "Value" "470uF 16V"
 			(at 218.44 90.5509 0)
 			(effects
@@
 			)
 		)
-		(property "Value" "2.2mH"
+		(property "Value" "470uF"
 			(at 189.738 86.106 90)
 			(effects
@@
 			)
 		)
-		(property "Footprint" "Package_SO:SOIC-8_3.9x4.9mm_P1.27mm"
+		(property "Footprint" "NosLib:LNK302PN-SOIC-8_3.9x4.9mm_P1.27mm"
 			(at 109.22 81.28 0)
 			(effects
@@
 		(lib_id "Diode:US1M")
 		(at 189.23 52.07 0)
-		(mirror y)
+		(mirror x)
 		(unit 1)
 		(exclude_from_sim no)
@@
 		(dnp no)
 		(property "Reference" "D401"
-			(at 189.23 45.72 0)
+			(at 189.23 58.42 0)
 			(effects
 				(font
@@
 		)
 		(property "Value" "US1M"
-			(at 189.23 48.26 0)
+			(at 189.23 55.88 0)
 			(effects
 				(font
@@
 		)
 		(property "Footprint" "Diode_SMD:D_SMA"
-			(at 189.23 56.515 0)
-			(effects
-				(font
+			(at 189.23 47.625 0)
+			(effects
+				(font
